File: PCB/_autosave-PCB.kicad_pcb (KiCad board)
At the start: 2 copper layers, 26 x 49 mm, 8 parts, among them IC1 MSPM0G3507SPTR, J1 ICS43434 Breakout, J2 MAX98357_Breakout, J4 LED_Header, J5 MSPM0 Programming Header, J6 USBC_Power_Breakout, U2 254

Commit message: pcb update
Parts:
- moved J6 39.8 mm to (155.5, 89.2)
- moved J1 21.1 mm to (142.7, 62.2), turned to 90 degrees
Changed lines of the file:
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@@
 	(footprint "Connector_PinSocket_1.00mm:PinSocket_1x06_P1.00mm_Vertical"
 		(layer "F.Cu")
-		(at 163.5696 59.3072)
+		(at 142.6624 62.23 90)
 		(descr "Through hole straight socket strip, 1x06, 1.00mm pitch, single row (https://gct.co/files/drawings/bc065.pdf), script generated")
 		(tags "Through hole socket strip THT 1x06 1.00mm single row")
 		(property "Reference" "J1"
-			(at -0.29 -2.25 0)
+			(at -0.29 -2.25 90)
 			(layer "F.SilkS")
 			(effects
@@
 		)
 		(property "Value" "ICS43434 Breakout"
-			(at -0.29 7.25 0)
+			(at -0.29 7.25 90)
 			(layer "F.Fab")
 			(effects
@@
 		)
 		(property "Datasheet" "~"
-			(at 0 0 0)
+			(at 0 0 90)
 			(layer "F.Fab")
 			(hide yes)
@@
 		)
 		(property "Description" "Generic connector, single row, 01x06, script generated"
-			(at 0 0 0)
+			(at 0 0 90)
 			(layer "F.Fab")
 			(hide yes)
@@
 		(attr through_hole)
 		(fp_line
+			(start 0.685 -0.81)
+			(end 0.685 0)
+			(stroke
+				(width 0.12)
+				(type solid)
+			)
+			(layer "F.SilkS")
+		)
+		(fp_line
+			(start 0 -0.81)
+			(end 0.685 -0.81)
+			(stroke
+				(width 0.12)
+				(type solid)
+			)
+			(layer "F.SilkS")
+		)
+		(fp_line
+			(start -1.1 0.5)
+			(end -0.685 0.5)
+			(stroke
+				(width 0.12)
+				(type solid)
+			)
+			(layer "F.SilkS")
+		)
+		(fp_line
 			(start -1.1 0.5)
 			(end -1.1 5.81)
@@
 		)
 		(fp_line
-			(start -1.1 0.5)
-			(end -0.685 0.5)
+			(start 0.52 1.445898)
+			(end 0.52 1.554102)
+			(stroke
+				(width 0.12)
+				(type solid)
+			)
+			(layer "F.SilkS")
+		)
+		(fp_line
+			(start 0.52 2.445898)
+			(end 0.52 2.554102)
+			(stroke
+				(width 0.12)
+				(type solid)
+			)
+			(layer "F.SilkS")
+		)
+		(fp_line
+			(start 0.52 3.445898)
+			(end 0.52 3.554102)
+			(stroke
+				(width 0.12)
+				(type solid)
+			)
+			(layer "F.SilkS")
+		)
+		(fp_line
+			(start 0.52 4.445898)
+			(end 0.52 4.554102)
+			(stroke
+				(width 0.12)
+				(type solid)
+			)
+			(layer "F.SilkS")
+		)
+		(fp_line
+			(start 0.52 5.445898)
+			(end 0.52 5.81)
 			(stroke
 				(width 0.12)
@@
 		)
 		(fp_line
-			(start 0 -0.81)
-			(end 0.685 -0.81)
-			(stroke
-				(width 0.12)
-				(type solid)
-			)
-			(layer "F.SilkS")
-		)
-		(fp_line
-			(start 0.52 1.445898)
-			(end 0.52 1.554102)
-			(stroke
-				(width 0.12)
-				(type solid)
-			)
-			(layer "F.SilkS")
-		)
-		(fp_line
-			(start 0.52 2.445898)
-			(end 0.52 2.554102)
-			(stroke
-				(width 0.12)
-				(type solid)
-			)
-			(layer "F.SilkS")
-		)
-		(fp_line
-			(start 0.52 3.445898)
-			(end 0.52 3.554102)
-			(stroke
-				(width 0.12)
-				(type solid)
-			)
-			(layer "F.SilkS")
-		)
-		(fp_line
-			(start 0.52 4.445898)
-			(end 0.52 4.554102)
-			(stroke
-				(width 0.12)
-				(type solid)
-			)
-			(layer "F.SilkS")
-		)
-		(fp_line
-			(start 0.52 5.445898)
-			(end 0.52 5.81)
-			(stroke
-				(width 0.12)
-				(type solid)
-			)
-			(layer "F.SilkS")
-		)
-		(fp_line
-			(start 0.685 -0.81)
-			(end 0.685 0)
-			(stroke
-				(width 0.12)
-				(type solid)
-			)
-			(layer "F.SilkS")
+			(start 0.96 -1.25)
+			(end 0.96 6.25)
+			(stroke
+				(width 0.05)
+				(type solid)
+			)
+			(layer "F.CrtYd")
 		)
 		(fp_line
@@
 		)
 		(fp_line
+			(start 0.96 6.25)
+			(end -1.54 6.25)
+			(stroke
+				(width 0.05)
+				(type solid)
+			)
+			(layer "F.CrtYd")
+		)
+		(fp_line
 			(start -1.54 6.25)
 			(end -1.54 -1.25)
@@
 		)
 		(fp_line
-			(start 0.96 -1.25)
-			(end 0.96 6.25)
-			(stroke
-				(width 0.05)
-				(type solid)
-			)
-			(layer "F.CrtYd")
-		)
-		(fp_line
-			(start 0.96 6.25)
-			(end -1.54 6.25)
-			(stroke
-				(width 0.05)
-				(type solid)
-			)
-			(layer "F.CrtYd")
+			(start 0.085 -0.75)
+			(end 0.46 -0.375)
+			(stroke
+				(width 0.1)
+				(type solid)
+			)
+			(layer "F.Fab")
 		)
 		(fp_line
@@
 		)
 		(fp_line
+			(start 0.46 -0.375)
+			(end 0.46 5.75)
+			(stroke
+				(width 0.1)
+				(type solid)
+			)
+			(layer "F.Fab")
+		)
+		(fp_line
+			(start 0.46 5.75)
+			(end -1.04 5.75)
+			(stroke
+				(width 0.1)
+				(type solid)
+			)
+			(layer "F.Fab")
+		)
+		(fp_line
 			(start -1.04 5.75)
 			(end -1.04 -0.75)
@@
 			(layer "F.Fab")
 		)
-		(fp_line
-			(start 0.085 -0.75)
-			(end 0.46 -0.375)
-			(stroke
-				(width 0.1)
-				(type solid)
-			)
-			(layer "F.Fab")
-		)
-		(fp_line
-			(start 0.46 -0.375)
-			(end 0.46 5.75)
-			(stroke
-				(width 0.1)
-				(type solid)
-			)
-			(layer "F.Fab")
-		)
-		(fp_line
-			(start 0.46 5.75)
-			(end -1.04 5.75)
-			(stroke
-				(width 0.1)
-				(type solid)
-			)
-			(layer "F.Fab")
-		)
 		(fp_text user "${REFERENCE}"
-			(at -0.29 2.5 90)
+			(at 0 0 0)
 			(layer "F.Fab")
 			(effects
@@
 		)
 		(pad "1" thru_hole rect
-			(at 0 0)
+			(at 0 0 90)
 			(size 0.85 0.85)
 			(drill 0.5)
@@
 		)
 		(pad "2" thru_hole circle
-			(at 0 1)
+			(at 0 1 90)
 			(size 0.85 0.85)
 			(drill 0.5)
@@
 		)
 		(pad "3" thru_hole circle
-			(at 0 2)
+			(at 0 2 90)
 			(size 0.85 0.85)
 			(drill 0.5)
@@
 		)
 		(pad "4" thru_hole circle
-			(at 0 3)
+			(at 0 3 90)
 			(size 0.85 0.85)
 			(drill 0.5)
@@
 		)
 		(pad "5" thru_hole circle
-			(at 0 4)
+			(at 0 4 90)
 			(size 0.85 0.85)
 			(drill 0.5)
@@
 		)
 		(pad "6" thru_hole circle
-			(at 0 5)
+			(at 0 5 90)
 			(size 0.85 0.85)
 			(drill 0.5)
@@
 	(footprint "SpinnyKitty:USBC_POWER_BREAKOUT"
 		(layer "F.Cu")
-		(at 118.6688 74.2696 180)
+		(at 155.5496 89.2048 180)
 		(property "Reference" "J6"
 			(at -3 -3.89 0)
@@
 		)
 		(property "Value" "MSPM0 Programming Header"
-			(at -3.3024 -12.518 0)
-			(layer "F.Fab")
-			(effects
+			(at 11.7348 1.8872 0)
+			(layer "F.Fab")
+			(effects
