File: PCB/PCB.kicad_sch (KiCad schematic)
At the start: 43 parts, among them IC1 MSPM0G3507SDGS28R, IC2 AP33771CFBZ-13-FA01, IC3 LT8609EMSE#PBF, IC4 AP63203WU-7, J1 ICS43434 Breakout, J2 MAX98357_Breakout, J3 UJ20-C-V-SMT-TR-68, J4 LED_Header, J5 MSPM0 Programming Header, J6 USBC_Power_Breakout, J8 Motor_Driver_Power, Q1 PSMN2R6-30YLC,115, Q2 PSMN2R6-30YLC,115, U2 254

Commit message: backup power rail pcb
Parts:
- added C14, C16, C18, C20, C23, C25, C26, C29, C31, C32: 0.1uF, Capacitor_SMD:C_0805_2012Metric_Pad1.18x1.45mm_HandSolder, symbol Device:C_Small
- added C15, C17, C21, C22, C24, C28, C30: 47uF, Capacitor_SMD:C_0805_2012Metric_Pad1.18x1.45mm_HandSolder, symbol Device:C_Small
- added C19, C27, C33: 22uF, Capacitor_SMD:C_1206_3216Metric_Pad1.33x1.80mm_HandSolder, symbol Device:C_Small
- added J7: ~, Connector_PinHeader_2.54mm:PinHeader_1x04_P2.54mm_Vertical, symbol SpinnyKitty:Power_Debug
- C13: value 100nF -> 0.1uF
- U4: footprint (none) -> SpinnyKitty:3V3 1.8A Buck
Connections:
- net +12V: now also C14.2, C15.2, C24.2, C25.2, J7.1 (12V)
- net +3V3: now also U4.2 (OUT+), C18.2, C19.2, C26.2, C27.2, C32.1, C33.1, J7.3 (3V3); no longer U2.7 (3V), U4.1 (IN+)
- net +5V: now also U2.8 (5V), U4.4 (IN+), C16.2, C17.2, C20.2, C21.2, C22.2, C23.2, C28.2, C29.2, C30.1, C31.1, J7.2 (5V); no longer U4.1 (IN+)
- net GND: now also U4.3 (IN-), C14.1, C15.1, C16.1, C17.1, C18.1, C19.1, C20.1, C21.1, C22.1, C23.1, C24.1, C25.1, C26.1, C27.1, C28.1, C29.1, C30.2, C31.2, C32.2, C33.2, J7.4 (GND)
Other:
- note added: "Compute"
- note added: "Peripherals"
- note added: "Power Debug"
- note added: "Power System Replacement Modules"
- moved on the sheet: IC1, J1, J2, J4, J5, J6, J8, U1, U2, U3, U4

Commit message: schematic update
Parts:
- added J9: ~, symbol SpinnyKitty:Motor_Driver_Control
Connections:
- net AMP_BCLK: now also U1.7 (GPIO26)
- net AMP_LRC: now also U1.8 (GPIO25)
- net GND: now also J9.4 (GND)
- net MTX_ERX: now reaches IC1.15 (PA10_/_CLK_OUT)
- net MTX_ERX: now also U1.21 (GPIO16)
- net ETX_MRX: now reaches IC1.16 (PA11)
- net ETX_MRX: now also U1.22 (GPIO17)
- net MD_ENA: now reaches IC1.25 (PA22_/_CLK_OUT_/_A0_7)
- net MD_ENA: now also J9.3 (ENA)
- net MD_IN2: now reaches IC1.27 (PA24_/_A0_3)
- net MD_IN2: now also J9.2 (IN2)
- net MD_IN1: now reaches IC1.28 (PA25_/_A0_2)
- net MD_IN1: now also J9.1 (IN1)
- net AMP_DIN: now reaches J2.5 (DIN)
- net AMP_DIN: now also U1.29 (GPIO22)
- net PWM_BU: now reaches U1.20 (GPIO4)
- no-connect marks 12 -> 14
Changed lines of the file:
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@@
 	)
 	(no_connect
+		(at 332.74 127)
+	)
+	(no_connect
 		(at 332.74 111.76)
 	)
@@
 	)
 	(no_connect
+		(at 332.74 124.46)
+	)
+	(no_connect
 		(at 78.74 185.42)
 	)
@@
 		)
 	)
+	(label "MD_ENA"
+		(at 163.83 110.49 0)
+		(effects
+			(font
+				(size 1.27 1.27)
+			)
+			(justify left bottom)
+		)
+	)
+	(label "ETX_MRX"
+		(at 34.29 72.39 180)
+		(effects
+			(font
+				(size 1.27 1.27)
+			)
+			(justify right bottom)
+		)
+	)
 	(label "GND"
 		(at 279.4 193.04 0)
@@
 		)
 	)
+	(label "MD_IN1"
+		(at 163.83 102.87 0)
+		(effects
+			(font
+				(size 1.27 1.27)
+			)
+			(justify left bottom)
+		)
+	)
 	(label "SD_CLK"
 		(at 294.64 73.66 180)
@@
 		)
 	)
+	(label "ETX_MRX"
+		(at 163.83 133.35 0)
+		(effects
+			(font
+				(size 1.27 1.27)
+			)
+			(justify left bottom)
+		)
+	)
+	(label "AMP_DIN"
+		(at 332.74 121.92 0)
+		(effects
+			(font
+				(size 1.27 1.27)
+			)
+			(justify left bottom)
+		)
+	)
 	(label "DP"
 		(at 78.74 180.34 0)
@@
 		)
 	)
+	(label "PWM_BU"
+		(at 34.29 67.31 180)
+		(effects
+			(font
+				(size 1.27 1.27)
+			)
+			(justify right bottom)
+		)
+	)
 	(label "GATE_DRV"
 		(at 189.23 184.15 0)
@@
 		)
 	)
+	(label "MTX_ERX"
+		(at 34.29 69.85 180)
+		(effects
+			(font
+				(size 1.27 1.27)
+			)
+			(justify right bottom)
+		)
+	)
 	(label "IC_CC2"
 		(at 78.74 177.8 0)
@@
 		)
 	)
+	(label "AMP_DIN"
+		(at 34.29 90.17 180)
+		(effects
+			(font
+				(size 1.27 1.27)
+			)
+			(justify right bottom)
+		)
+	)
 	(label "AMP_BCLK"
 		(at 332.74 119.38 0)
@@
 		)
 	)
+	(label "AMP_BCLK"
+		(at 62.23 72.39 0)
+		(effects
+			(font
+				(size 1.27 1.27)
+			)
+			(justify left bottom)
+		)
+	)
 	(label "GATE_DRV"
 		(at 190.5 201.93 0)
@@
 		)
 	)
+	(label "MTX_ERX"
+		(at 163.83 135.89 0)
+		(effects
+			(font
+				(size 1.27 1.27)
+			)
+			(justify left bottom)
+		)
+	)
 	(label "GND"
 		(at 107.95 205.74 270)
@@
 		)
 	)
+	(label "MD_ENA"
+		(at 368.3 69.85 180)
+		(effects
+			(font
+				(size 1.27 1.27)
+			)
+			(justify right bottom)
+		)
+	)
 	(label "5V"
 		(at 215.9 170.18 180)
@@
 		)
 	)
+	(label "MD_IN2"
+		(at 368.3 67.31 180)
+		(effects
+			(font
+				(size 1.27 1.27)
+			)
+			(justify right bottom)
+		)
+	)
 	(label "5V"
 		(at 306.07 218.44 180)
@@
 		)
 	)
+	(label "AMP_LRC"
+		(at 62.23 74.93 0)
+		(effects
+			(font
+				(size 1.27 1.27)
+			)
+			(justify left bottom)
+		)
+	)
 	(label "DN"
 		(at 139.7 187.96 0)
@@
 		)
 	)
+	(label "MD_IN2"
+		(at 163.83 105.41 0)
+		(effects
+			(font
+				(size 1.27 1.27)
+			)
+			(justify left bottom)
+		)
+	)
 	(label "GND"
 		(at 307.34 162.56 0)
@@
 		)
 	)
+	(label "MD_IN1"
+		(at 368.3 64.77 180)
+		(effects
+			(font
+				(size 1.27 1.27)
+			)
+			(justify right bottom)
+		)
+	)
 	(label "GND"
 		(at 382.27 226.06 270)
@@
 		)
 	)
+	(label "GND"
+		(at 368.3 72.39 180)
+		(effects
+			(font
+				(size 1.27 1.27)
+			)
+			(justify right bottom)
+		)
+	)
 	(label "IC_CC1"
 		(at 45.72 182.88 180)
@@
 		(exclude_from_sim no)
 		(in_bom yes)
-		(on_board no)
+		(on_board yes)
 		(dnp no)
 		(fields_autoplaced yes)
@@
 		(exclude_from_sim no)
 		(in_bom no)
-		(on_board no)
+		(on_board yes)
 		(dnp no)
 		(fields_autoplaced yes)
@@
 		(exclude_from_sim no)
 		(in_bom no)
-		(on_board no)
+		(on_board yes)
 		(dnp no)
 		(fields_autoplaced yes)
@@
 		(exclude_from_sim no)
 		(in_bom no)
-		(on_board no)
+		(on_board yes)
 		(dnp no)
 		(property "Reference" "J5"
@@
 					(unit 1)
 				)
+			)
+		)
+	)
+	(symbol
+		(lib_id "SpinnyKitty:Motor_Driver_Control")
+		(at 373.38 68.58 0)
+		(unit 1)
+		(exclude_from_sim no)
+		(in_bom yes)
+		(on_board yes)
+		(dnp no)
+		(fields_autoplaced yes)
+		(property "Reference" "J9"
+			(at 377.19 67.3099 0)
+			(effects
+				(font
+					(size 1.27 1.27)
+				)
+				(justify left)
+			)
+		)
+		(property "Value" "~"
+			(at 377.19 69.8499 0)
+			(effects
+				(font
+					(size 1.27 1.27)
+				)
+				(justify left)
+			)
+		)
+		(property "Footprint" ""
+			(at 373.38 68.58 0)
+			(effects
+				(font
+					(size 1.27 1.27)
+				)
+				(hide yes)
+			)
+		)
+		(property "Datasheet" ""
+			(at 373.38 68.58 0)
+			(effects
+				(font
+					(size 1.27 1.27)
+				)
+				(hide yes)
+			)
+		)
+		(property "Description" ""
+			(at 373.38 68.58 0)
+			(effects
+				(font
+					(size 1.27 1.27)
+				)
+				(hide yes)
+			)
+		)
+		(pin "4"
+		)
+		(pin "3"
+		)
+		(pin "2"
+		)
+		(pin "1"
+		)
+		(instances
+			(project ""
+				(path "/954dff68-cc85-452c-9053-ce35508878d2"
+					(reference "J9")
+					(unit 1)
+				)

Commit message: schematic update
Parts:
- removed C33: 22uF, Capacitor_SMD:C_1206_3216Metric_Pad1.33x1.80mm_HandSolder, symbol Device:C_Small
- added R12, R13: 2.2k, Resistor_SMD:R_0603_1608Metric_Pad0.98x0.95mm_HandSolder, symbol Device:R_Small_US
- added R14, R15, R16, R17, R18, R19, R20, R21: 10k, Resistor_SMD:R_0603_1608Metric_Pad0.98x0.95mm_HandSolder, symbol Device:R_Small_US
- added S1, S2, S3, S4, S5, S6, S7, S8: TL3305AF260QG, TL3305AF160QG, symbol TL3305AF260QG:TL3305AF260QG
- C21, C22: value 47uF -> 4.7uF; Mouser Part Number 810-C3216X5R1E476M -> KGM21AR71E475KU; Mouser Price/Stock https://mou.sr/3ZlIJTu -> https://mou.sr/41nY4qi
- C27: value 22uF -> 4.7uF; footprint Capacitor_SMD:C_1206_3216Metric_Pad1.33x1.80mm_HandSolder -> Capacitor_SMD:C_0805_2012Metric_Pad1.18x1.45mm_HandSolder; Mouser Part Number 963-MSASE31LBB7226MT -> KGM21AR71E475KU; Mouser Price/Stock https://mou.sr/4mnXr9C -> https://mou.sr/41nY4qi
- C28: value 47uF -> 22uF; footprint Capacitor_SMD:C_0805_2012Metric_Pad1.18x1.45mm_HandSolder -> Capacitor_SMD:C_1206_3216Metric_Pad1.33x1.80mm_HandSolder; Mouser Part Number 810-C3216X5R1E476M -> 963-MSASE31LBB7226MT; Mouser Price/Stock https://mou.sr/3ZlIJTu -> https://mou.sr/4mnXr9C
- C30: value 47uF -> 10uF; footprint Capacitor_SMD:C_0805_2012Metric_Pad1.18x1.45mm_HandSolder -> Capacitor_SMD:C_1206_3216Metric_Pad1.33x1.80mm_HandSolder; Mouser Part Number 810-C3216X5R1E476M -> 963-BAST31LAB7106KT; Mouser Price/Stock https://mou.sr/3ZlIJTu -> https://mou.sr/4hqfbil
- C4: Mouser Part Number 581-KGM21AR71E105JU -> KGM21AR71E475KU
- J9: footprint (none) -> Connector_PinHeader_2.54mm:PinHeader_1x04_P2.54mm_Vertical
Connections:
- net +3V3: now also C27.1, R12.1, R13.1, R14.1, R15.1, R16.1, R17.1, R18.1, R19.1, R20.1, R21.1; no longer C27.2
- net +5V: now also C30.2; no longer C30.1
- net AMP_DIN: now also U1.6 (GPIO27); no longer U1.29 (GPIO22)
- net GND: now also C27.2, C30.1, J1.1 (SEL), U1.17 (GND), S1.1, S1.2, S2.1, S2.2, S3.1, S3.2, S4.1, S4.2, S5.1, S5.2, S6.1, S6.2, S7.1, S7.2, S8.1, S8.2; no longer C27.1, C30.2
- net BTN_LED: now reaches IC1.20 (PA17_/_A1_2)
- net BTN_LED: now also S8.3
- net BTN_MTR: now reaches IC1.21 (PA18_/_A1_3)
- net BTN_MTR: now also S7.3
- net SDA: now reaches IC1.4 (PA0)
- net SDA: now also U1.26 (GPIO21), R12.2
- net SCL: now reaches IC1.5 (PA1)
- net SCL: now also U1.29 (GPIO22), R13.2
- net MIC_LRCL: now reaches J1.2 (LRCL)
- net MIC_LRCL: now also U1.18 (GPIO15)
- net MIC_DOUT: now reaches J1.3 (DOUT)
- net MIC_DOUT: now also U1.10 (GPIO32)
- net MIC_BCLK: now reaches J1.4 (BCLK)
- net MIC_BCLK: now also U1.5 (GPIO14)
- net BTN_NXT: now reaches U1.11 (GPIO35)
- net BTN_NXT: now also S4.3
- net BTN_PRV: now reaches U1.12 (GPIO34)
- net BTN_PRV: now also S3.3
- net BTN_VDWN: now reaches U1.13 (GPIO39)
- net BTN_VDWN: now also S6.3
- net BTN_VUP: now reaches U1.14 (GPIO36)
- net BTN_VUP: now also S5.3
- net BTN_SP: now reaches U1.3 (GPIO13)
- net BTN_SP: now also S1.3
- net BTN_PP: now reaches U1.9 (GPIO33)
- net BTN_PP: now also S2.3
- new net: R17.2, S4.4
- new net: R14.2, S1.4
- new net: R21.2, S8.4
- new net: R20.2, S7.4
- new net: R16.2, S3.4
- new net: R19.2, S6.4
- new net: R15.2, S2.4
- new net: R18.2, S5.4
- no-connect marks 14 -> 20
Other:
- moved on the sheet: C32, J1

Commit message: complete pcb
Parts:
- added C33: 22uF, Capacitor_SMD:C_1206_3216Metric_Pad1.33x1.80mm_HandSolder, symbol Device:C_Small
- added C34: 0.1uF, Capacitor_SMD:C_0805_2012Metric_Pad1.18x1.45mm_HandSolder, symbol Device:C_Small
- added U5: SN74AHCT125N, SpinnyKitty:DIP794W45P254L1930H508Q14, symbol SN74AHCT125N:SN74AHCT125N
- renumbered C28 to C27, C29 to C28, C30 to C29, C31 to C30, C27 to C31
Connections:
- net +5V: now also C33.2, C34.2, U5.14 (VCC)
- net GND: now also C33.1, C34.1, U5.1 (1~{OE}), U5.7 (GND)
- net LED_DATA: now also IC1.18 (PA15_/_A1_0), U5.2 (1A); no longer J4.2 (DATA)
- new net LED_SHIFTED: J4.2 (DATA), U5.3 (1Y)
- no-connect marks 20 -> 29
Other:
- moved on the sheet: C22, C23, U2

Commit message: mspm0 update
Parts:
- added C35: 10uF, Capacitor_SMD:C_1206_3216Metric_Pad1.33x1.80mm_HandSolder, symbol Device:C_Small
- added C36: 10nF, Capacitor_SMD:C_0805_2012Metric_Pad1.18x1.45mm_HandSolder, symbol Device:C_Small
- added C37: 0.47uF, Capacitor_SMD:C_0805_2012Metric_Pad1.18x1.45mm_HandSolder, symbol Device:C_Small
- added R22: 47k, Resistor_SMD:R_0603_1608Metric_Pad0.98x0.95mm_HandSolder, symbol Device:R_Small_US
Connections:
- net +3V3: now also C35.1, R22.1
- net GND: now also C35.2, C36.1, C37.1
- net NRST: now also C36.2, R22.2
- net VCORE: now reaches IC1.3 (VCORE)
- net VCORE: now also C37.2
- no-connect marks 29 -> 41
Other:
- moved on the sheet: R12, R13
