File: PCB/PCB.kicad_sch (KiCad schematic)
At the start: 89 parts, among them IC1 MSPM0G3507SDGS28R, IC2 AP33771CFBZ-13-FA01, IC3 LT8609EMSE#PBF, IC4 AP63203WU-7, J1 ICS43434 Breakout, J2 MAX98357_Breakout, J3 UJ20-C-V-SMT-TR-68, J4 LED_Header, J5 MSPM0 Programming Header, J6 USBC_Power_Breakout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

Commit message: pcb backups
Parts:
- added R23: 100k, Resistor_SMD:R_0805_2012Metric_Pad1.20x1.40mm_HandSolder, symbol Device:R_Small_US
Connections:
- net GND: now also R23.2
- net at IC1.9 (PA2_/_ROSC): now also R23.1
Other:
- moved on the sheet: C37
Changed lines of the file:
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@@
 	)
 	(no_connect
+		(at 123.19 156.21)
+	)
+	(no_connect
 		(at 87.63 102.87)
 	)
@@
 	)
 	(no_connect
-		(at 87.63 123.19)
-	)
-	(no_connect
 		(at 332.74 127)
 	)
@@
 	(wire
 		(pts
+			(xy 87.63 123.19) (xy 83.82 123.19)
+		)
+		(stroke
+			(width 0)
+			(type default)
+		)
+	)
+	(wire
+		(pts
 			(xy 231.14 224.79) (xy 233.68 224.79)
 		)
@@
 	(wire
 		(pts
+			(xy 83.82 123.19) (xy 83.82 130.81)
+		)
+		(stroke
+			(width 0)
+			(type default)
+		)
+	)
+	(wire
+		(pts
 			(xy 297.18 179.07) (xy 304.8 179.07)
 		)
@@
 	(wire
 		(pts
+			(xy 83.82 130.81) (xy 77.47 130.81)
+		)
+		(stroke
+			(width 0)
+			(type default)
+		)
+	)
+	(wire
+		(pts
 			(xy 72.39 118.11) (xy 87.63 118.11)
 		)
@@
 	)
 	(label "GND"
-		(at 71.12 138.43 270)
+		(at 59.69 137.16 270)
 		(effects
 			(font
@@
 	)
 	(label "VCORE"
-		(at 71.12 133.35 180)
+		(at 59.69 132.08 180)
 		(effects
 			(font
@@
 	)
 	(label "GND"
+		(at 77.47 135.89 270)
+		(effects
+			(font
+				(size 1.27 1.27)
+			)
+			(justify right bottom)
+		)
+	)
+	(label "GND"
 		(at 196.85 109.22 180)
 		(effects
@@
 	(symbol
 		(lib_id "Device:R_Small_US")
+		(at 77.47 133.35 0)
+		(unit 1)
+		(exclude_from_sim no)
+		(in_bom yes)
+		(on_board yes)
+		(dnp no)
+		(fields_autoplaced yes)
+		(property "Reference" "R23"
+			(at 80.01 132.0799 0)
+			(effects
+				(font
+					(size 1.27 1.27)
+				)
+				(justify left)
+			)
+		)
+		(property "Value" "100k"
+			(at 80.01 134.6199 0)
+			(effects
+				(font
+					(size 1.27 1.27)
+				)
+				(justify left)
+			)
+		)
+		(property "Footprint" "Resistor_SMD:R_0805_2012Metric_Pad1.20x1.40mm_HandSolder"
+			(at 77.47 133.35 0)
+			(effects
+				(font
+					(size 1.27 1.27)
+				)
+				(hide yes)
+			)
+		)
+		(property "Datasheet" "~"
+			(at 77.47 133.35 0)
+			(effects
+				(font
+					(size 1.27 1.27)
+				)
+				(hide yes)
+			)
+		)
+		(property "Description" "Resistor, small US symbol"
+			(at 77.47 133.35 0)
+			(effects
+				(font
+					(size 1.27 1.27)
+				)
+				(hide yes)
+			)
+		)
+		(property "Mouser Part Number" "708-RNCF0805TKT100K"
+			(at 77.47 133.35 0)
+			(effects
+				(font
+					(size 1.27 1.27)
+				)
+				(justify left top)
+				(hide yes)
+			)
+		)
+		(property "Mouser Price/Stock" "https://mou.sr/4c6uqfk"
+			(at 77.47 133.35 0)
+			(effects
+				(font
+					(size 1.27 1.27)
+				)
+				(justify left top)
+				(hide yes)
+			)
+		)
+		(pin "2"
+		)
+		(pin "1"
+		)
+		(instances
+			(project "PCB"
+				(path "/954dff68-cc85-452c-9053-ce35508878d2"
+					(reference "R23")
+					(unit 1)
+				)
+			)
+		)
+	)
+	(symbol
+		(lib_id "Device:R_Small_US")
 		(at 255.27 104.14 0)
 		(unit 1)
@@
 	(symbol
 		(lib_id "Device:C_Small")
-		(at 71.12 135.89 180)
+		(at 59.69 134.62 180)
 		(unit 1)
 		(exclude_from_sim no)
@@
 		(fields_autoplaced yes)
 		(property "Reference" "C37"
-			(at 73.66 134.6135 0)
+			(at 62.23 133.3435 0)
 			(effects
 				(font
@@
 		)
 		(property "Value" "0.47uF"
-			(at 73.66 137.1535 0)
+			(at 62.23 135.8835 0)
 			(effects
 				(font
@@
 		)
 		(property "Footprint" "Capacitor_SMD:C_0805_2012Metric_Pad1.18x1.45mm_HandSolder"
-			(at 71.12 135.89 0)
+			(at 59.69 134.62 0)
 			(effects
 				(font
@@
 		)
 		(property "Datasheet" "~"
-			(at 71.12 135.89 0)
+			(at 59.69 134.62 0)
 			(effects
 				(font
@@
 		)
 		(property "Description" "Unpolarized capacitor, small symbol"
-			(at 71.12 135.89 0)
+			(at 59.69 134.62 0)
 			(effects
 				(font
@@
 		)
 		(property "Mouser Part Number" "581-08055C474K4T4A"
-			(at 71.12 135.89 90)
+			(at 59.69 134.62 90)
 			(effects
 				(font
@@
 		)
 		(property "Mouser Price/Stock" "https://mou.sr/4mquvOw"
-			(at 71.12 135.89 90)
+			(at 59.69 134.62 90)
 			(effects
 				(font
